File: Kicad/AURORAV1.kicad_sch (KiCad schematic)
At the start: 100 parts, among them J1 DX07S016JA1R1500, J2 DM3CS-SF, J3 TC2030-IDC-NL, J4 BAT_CONN, Q101 AO3401A, SW1 SW_SPDT, U1 RT8259GJ6, U10 RFM96W-433S2, U11 EDGE_ANTENNA, U12 USBLC6-2SC6, U2 STM32F446RET6, U3 H3LIS200DLTR, U4 MPL3115A2, U5 HDC1080, U6 LIS3MDL, U7 BMI270, U8 I3G4250DTR, U9 W25N01GVZEIG_TR, Y1 16MHz

Commit message: Updated Schematic/PCB Descriptions
Other:
- title: Log(er) -> AURORA
Changed lines of the file:
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@@
   (paper "A3")
   (title_block
-    (title "Log(er)")
-    (date "2022-12-05")
-    (rev "v0.1")
+    (title "AURORA")
+    (date "2023-01-07")
+    (rev "V1")
     (company "Balthazar Avionics")
   )
